File: usb-phy.kicad_sch (KiCad schematic)
At the start: 124 parts, among them J12 614004184726, J13 USB4105-GF-A, J14 USB4105-GF-A, Q17 BSS138PW, U15 NCP718BSN330T1G, U16 TPD4E05U06QDQARQ1, U17 TPD4E05U06QDQARQ1, U18 SN74HC595B, U19 MAX3421EETJ+, U20 FT4232H-56Q, U21 TPD4E05U06QDQARQ1, U22 TXU0304BQAR, U23 TXU0304BQAR, U24 TXU0304BQAR, U25 TUSB1106RSVR, U30 AP22615, U43 AP22615, U48 74LVC1T45GM, Y1 ABM8G-12.000MHZ-18-D2Y-T, Y2 ABM8G-12.000MHZ-18-D2Y-T

Commit message: Updated all symbols causing warnings with no signal connected to pad, added thermal vias on level shifters' thermal pad with small tweaks on signal routing near this area
Connections:
- net GND: now also U22.15 (GND), U23.15 (GND), U24.15 (GND)
Changed lines of the file:
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@@
     (pin "13")
     (pin "14")
+    (pin "15")
     (pin "2")
     (pin "3")
@@
     (pin "2")
     (pin "3")
+    (pin "4")
     (pin "5")
   )
@@
     (pin "1")
   )
-  (symbol (lib_id "K410T-devboard:TXU0304BQAR") (at 322.58 181.61 0) (unit 1)
+  (symbol (lib_name "TXU0304BQAR_2") (lib_id "K410T-devboard:TXU0304BQAR") (at 322.58 181.61 0) (unit 1)
     (in_bom yes) (on_board yes)
     (property "Reference" "U23" (id 0) (at 329.565 189.23 0)
@@
     (pin "13")
     (pin "14")
+    (pin "15")
     (pin "2")
     (pin "3")
@@
     (pin "1")
   )
-  (symbol (lib_id "K410T-devboard:TXU0304BQAR") (at 322.58 214.63 0) (unit 1)
+  (symbol (lib_name "TXU0304BQAR_1") (lib_id "K410T-devboard:TXU0304BQAR") (at 322.58 214.63 0) (unit 1)
     (in_bom yes) (on_board yes)
     (property "Reference" "U24" (id 0) (at 329.565 222.25 0)
@@
     (pin "13")
     (pin "14")
+    (pin "15")
     (pin "2")
     (pin "3")
